File: Keyboard/Keyboard.kicad_pcb (KiCad board)
At the start: 2 copper layers, 344.6 x 135 mm, 129 parts, among them SW1 ESC_(1,1), SW10 LWin_(5,2), SW11 #2_(1,3), SW12 W_(2,3), SW13 S_(3,3), SW14 X_(4,3), SW15 LAlt_(5,3), SW16 #3_(1,4), SW17 E_(2,4), SW18 D_(3,4), SW19 C_(4,4), SW2 Tab_(2,1), SW20 #4_(1,5), SW21 R_(2,5), SW22 F_(3,5), SW23 V_(4,5), SW24 #5_(1,6), SW25 T_(2,6), SW26 G_(3,6), SW27 B_(4,6), SW28 Space_(5,6), SW29 #6_(1,7), SW3 CapsLock_(3,1), SW30 Y_(2,7), SW31 H_(3,7), SW32 N_(4,7), SW33 #7_(1,8), SW34 U_(2,8), SW35 J_(3,8), SW36 M_(4,8), SW37 #8_(1,9), SW38 I_(2,9), SW39 K_(3,9), SW4 Shift_(4,1), SW40 <,_(4,9), SW41 RAlt_(5,9), SW42 #9_(1,10), SW43 O_(2,10), SW44 L_(3,10), SW45 >._(4,10), SW46 RWin_(5,10), SW47 #0_(1,11), SW48 P_(2,11), SW49 :;_(3,11), SW5 LCtrl_(5,1), SW50 ?/_(4,11), SW51 Menu_(5,11), SW52 '-'_(1,12), SW53 {_(2,12), SW54 "'_(3,12), SW55 ShiftR_(4,12), SW56 RCtrl_(5,12), SW57 '+'_(1,13), SW58 }_(2,13), SW59 Enter_(3,13), SW6 #1_(1,2), SW60 Backspace_(1,14), SW61 |_(2,14), SW7 Q_(2,2), SW8 A_(3,2), SW9 Z_(4,2), U2 RP2040

Commit message: Rework layout: flip switches, clear routing, place diodes under switches
- Flip all 61 MX hot-swap footprints so sockets sit on the bottom (B.Cu)
  per the MX_V2 library's 2024 change; pin holes now match standard MX
- Delete all tracks and vias for a full reroute
- Move each diode to the bottom side, 5 mm below its switch's stem
- Remove GND fills on both layers (not needed for the matrix)

Co-Authored-By: Claude Opus 5.5 <noreply@anthropic.com>
Claude-Session: https://claude.ai/code/session_01TWtb48LXBV9JFeuN4caNHj
Parts:
- SW1, SW10, SW11, SW12, SW13, SW14, SW15, SW16, SW17, SW18, SW19, SW2, SW20, SW21, SW22, SW23, SW24, SW25, SW26, SW27, SW28, SW29, SW3, SW30, SW31, SW32, SW33, SW34, SW35, SW36, SW37, SW38, SW39, SW4, SW40, SW41, SW42, SW43, SW44, SW45, SW46, SW47, SW48, SW49, SW5, SW50, SW51, SW52, SW53, SW54, SW55, SW56, SW57, SW58, SW59, SW6, SW60, SW61, SW7, SW8, SW9: moved to B.Cu
- moved D7 86.9 mm to (193.4, 87.9), turned to 180 degrees
- moved D8 86.4 mm to (212.4, 87.9), turned to 180 degrees
- moved D5 86.4 mm to (155.3, 87.9), turned to 180 degrees
- moved D9 86.3 mm to (231.5, 87.9), turned to 180 degrees
- moved D4 86.0 mm to (136.2, 87.9), turned to 180 degrees
- moved D6 85.8 mm to (174.3, 87.9), turned to 180 degrees
- moved D10 85.5 mm to (250.5, 87.9), turned to 180 degrees
- moved D3 85.2 mm to (117.2, 87.9), turned to 180 degrees
- moved D11 85.2 mm to (269.6, 87.9), turned to 180 degrees
- moved D12 84.8 mm to (288.6, 87.9), turned to 180 degrees
- moved D13 84.6 mm to (307.7, 87.9), turned to 180 degrees
- moved D1 83.7 mm to (79.1, 87.9), turned to 180 degrees
- moved D2 83.5 mm to (98.1, 87.9), turned to 180 degrees
- moved D14 83.3 mm to (336.2, 87.9), turned to 180 degrees
- moved D21 67.2 mm to (202.9, 107.0), turned to 180 degrees
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Routing:
- net Row 4: track 405.4 -> 0.00 mm
- net Row 3: track 403.5 -> 0.00 mm
- net Row 5: track 403.1 -> 0.00 mm
- net Column 1: track 389.4 -> 0.00 mm, vias 3 -> 0
- net Row 1: track 384.2 -> 0.00 mm
- net Row 2: track 375.2 -> 0.00 mm
- net Column 2: track 353.3 -> 0.00 mm, vias 3 -> 0
- net Column 3: track 328.5 -> 0.00 mm, vias 3 -> 0
- net Column 4: track 290.9 -> 0.00 mm, vias 3 -> 0
- net Column 6: track 278.4 -> 0.00 mm, vias 3 -> 0
- net Column 5: track 268.3 -> 0.00 mm, vias 3 -> 0
- net Column 7: track 251.2 -> 0.00 mm, vias 3 -> 0
- net Column 8: track 235.4 -> 0.00 mm, vias 3 -> 0
- net Column 9: track 229.7 -> 0.00 mm, vias 4 -> 0
- net Column 10: track 218.8 -> 0.00 mm, vias 4 -> 0
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- removed copper zone on B.Cu, net GND
- removed copper zone on F.Cu, net GND
